File: KiCAD/MCU.sch (KiCad schematic (older format))
At the start: 0 parts

Commit message: Add mcu
Parts:
- added U?: STM32F411CEUx, Package_DFN_QFN:QFN-48-1EP_7x7mm_P0.5mm_EP5.6x5.6mm, symbol MCU_ST_STM32F4:STM32F411CEUx
Changed lines of the file:
@@
 $Descr A4 11693 8268
 encoding utf-8
-Sheet 1 5
+Sheet 3 6
 Title "AM & FM Transceiver"
 Date ""
@@
 Comment4 ""
 $EndDescr
+$Comp
+L MCU_ST_STM32F4:STM32F411CEUx U?
+U 1 1 5E7EE1B1
+P 5350 3150
+F 0 "U?" H 5300 4831 50  0000 C CNN
+F 1 "STM32F411CEUx" H 5300 4740 50  0000 C CNN
+F 2 "Package_DFN_QFN:QFN-48-1EP_7x7mm_P0.5mm_EP5.6x5.6mm" H 4750 1650 50  0001 R CNN
+F 3 "http://www.st.com/st-web-ui/static/active/en/resource/technical/document/datasheet/DM00115249.pdf" H 5350 3150 50  0001 C CNN
+	1    5350 3150
+	1    0    0    -1
+$EndComp
 $EndSCHEMATC
