File: KiCAD/Si5351_Filter.sch (KiCad schematic (older format))
At the start: 4 parts

Commit message: Just save files Begin PCB
Parts:
- C1, C2: renamed from C?; footprint (none) -> Capacitor_SMD:C_0805_2012Metric
- R3, R4: renamed from R?; footprint (none) -> Resistor_SMD:R_0805_2012Metric
Changed lines of the file:
@@
 $Descr A4 11693 8268
 encoding utf-8
-Sheet 2 5
+Sheet 2 4
 Title "AM & FM Transceiver"
 Date ""
@@
 Clk0_Fo
 $Comp
-L Device:C C?
+L Device:C C2
 U 1 1 5E724D9F
 P 4000 1100
-F 0 "C?" V 3748 1100 50  0000 C CNN
+F 0 "C2" V 3748 1100 50  0000 C CNN
 F 1 "100n" V 3839 1100 50  0000 C CNN
-F 2 "" H 4038 950 50  0001 C CNN
+F 2 "Capacitor_SMD:C_0805_2012Metric" H 4038 950 50  0001 C CNN
 F 3 "~" H 4000 1100 50  0001 C CNN
 	1    4000 1100
@@
 $EndComp
 $Comp
-L Device:R R?
+L Device:R R3
 U 1 1 5E725253
 P 3600 1100
-F 0 "R?" V 3393 1100 50  0000 C CNN
+F 0 "R3" V 3393 1100 50  0000 C CNN
 F 1 "100" V 3484 1100 50  0000 C CNN
-F 2 "" V 3530 1100 50  0001 C CNN
+F 2 "Resistor_SMD:R_0805_2012Metric" V 3530 1100 50  0001 C CNN
 F 3 "~" H 3600 1100 50  0001 C CNN
 	1    3600 1100
@@
 $EndComp
 $Comp
-L Device:R R?
+L Device:R R4
 U 1 1 5E725401
 P 3800 1300
-F 0 "R?" H 3870 1346 50  0000 L CNN
+F 0 "R4" H 3870 1346 50  0000 L CNN
 F 1 "100" H 3870 1255 50  0000 L CNN
-F 2 "" V 3730 1300 50  0001 C CNN
+F 2 "Resistor_SMD:R_0805_2012Metric" V 3730 1300 50  0001 C CNN
 F 3 "~" H 3800 1300 50  0001 C CNN
 	1    3800 1300
@@
 $EndComp
 $Comp
-L power:GND #PWR?
+L power:GND #PWR0123
 U 1 1 5E726822
 P 3800 1550
-F 0 "#PWR?" H 3800 1300 50  0001 C CNN
+F 0 "#PWR0123" H 3800 1300 50  0001 C CNN
 F 1 "GND" H 3805 1377 50  0000 C CNN
 F 2 "" H 3800 1550 50  0001 C CNN
@@
 	2950 1100 3050 1100
 $Comp
-L Device:C C?
+L Device:C C1
 U 1 1 5E7270D7
 P 3200 1100
-F 0 "C?" V 2948 1100 50  0000 C CNN
+F 0 "C1" V 2948 1100 50  0000 C CNN
 F 1 "100n" V 3039 1100 50  0000 C CNN
-F 2 "" H 3238 950 50  0001 C CNN
+F 2 "Capacitor_SMD:C_0805_2012Metric" H 3238 950 50  0001 C CNN
 F 3 "~" H 3200 1100 50  0001 C CNN
 	1    3200 1100
