File: KiCAD/AM Module.sch (KiCad schematic (older format))
At the start: 16 parts

Commit message: Add mcu
Parts:
- removed U?: LM321, Package_TO_SOT_SMD:SOT-23-5, symbol Amplifier_Operational:LM321
- added U?: AD8001AN, Package_DIP:DIP-8_W7.62mm, symbol Amplifier_Operational:AD8001AN
Changed lines of the file:
@@
 $Descr A4 11693 8268
 encoding utf-8
-Sheet 5 5
+Sheet 4 6
 Title "AM & FM Transceiver"
 Date ""
@@
 	0    1    1    0
 $EndComp
-$Comp
-L Amplifier_Operational:LM321 U?
-U 1 1 5E77E0AD
-P 5650 2800
-AR Path="/5E77AF45/5E77E0AD" Ref="U?"  Part="1"
-AR Path="/5E7940EB/5E77E0AD" Ref="U?"  Part="1"
-F 0 "U?" H 5994 2846 50  0000 L CNN
-F 1 "LM321" H 5994 2755 50  0000 L CNN
-F 2 "Package_TO_SOT_SMD:SOT-23-5" H 5650 2800 50  0001 C CNN
-F 3 "http://www.ti.com/lit/ds/symlink/lm321.pdf" H 5650 2800 50  0001 C CNN
-	1    5650 2800
-	1    0    0    -1
-$EndComp
 Wire Wire Line
 	5350 2700 4800 2700
@@
 Wire Wire Line
 	4200 3050 4100 3050
+$Comp
+L Amplifier_Operational:AD8001AN U?
+U 1 1 5E7C4873
+P 5650 2800
+F 0 "U?" H 5650 2950 50  0000 L CNN
+F 1 "AD8001AN" H 5650 2650 50  0000 L CNN
+F 2 "Package_DIP:DIP-8_W7.62mm" H 5550 2600 50  0001 L CNN
+F 3 "https://www.analog.com/media/en/technical-documentation/data-sheets/ad8001.pdf" H 5800 2950 50  0001 C CNN
+	1    5650 2800
+	1    0    0    -1
+$EndComp
 $EndSCHEMATC

Commit message: Add MCU module and other modules
Other:
- note added: "bc557?"
Changed lines of the file:
@@
 $Descr A4 11693 8268
 encoding utf-8
-Sheet 4 6
+Sheet 4 5
 Title "AM & FM Transceiver"
 Date ""
@@
 	1    0    0    -1
 $EndComp
+Text Notes 6750 3300 0    50   ~ 0
+bc557?
 $EndSCHEMATC

Commit message: Just save files Begin PCB
Parts:
- removed R? (x4): R, symbol Device:R
- added U3: MCP4651, Package_SO:TSSOP-14_4.4x5mm_P0.65mm, symbol SA612A:MCP4651
- C3, C4: renamed from C?; footprint (none) -> Capacitor_SMD:C_0805_2012Metric
- Q1, Q3: renamed from Q?; footprint Package_TO_SOT_THT:TO-39-3 -> Package_TO_SOT_THT:TO-92L_Inline_Wide
- Q2: renamed from Q?; footprint Package_TO_SOT_THT:TO-92_Inline -> Package_TO_SOT_THT:TO-92_Inline_Wide
- R13, R14, R5, R6, R7, R8: renamed from R?; footprint (none) -> Resistor_SMD:R_0805_2012Metric
- gave numbers to parts that had none: 1
Connections:
- net +12V is gone; now on net +5V: Q1.3 (C), U2.7 (V+)
- net +5V: now also U3.10 (P0B), U3.14 (VDD)
- net Feed_BackBFin: now also U3.9 (P0W)
- net GND: now also U3.1 (A0/HVC), U3.12 (A2), U3.13 (A1), U3.4 (Vss), U3.7 (P1A), U3.8 (P0A)
- net H1: now reaches Q1.1 (E), Q2.1 (E), Q3.3 (C), R13.1, R8.2
- net H1: now also U3.5 (P1B)
- net W1: now reaches U2.2 (-)
- net W1: now also U3.6 (P1W)
- new net DS_SCL: U3.2 (SCL)
- new net DS_SDA: U3.3 (SDA)

Commit message: Make PCB and change NPN and PNP for AM output
Parts:
- removed Q3: 2N2219, Package_TO_SOT_THT:TO-92L_Inline_Wide, symbol Transistor_BJT:2N2219
- removed U2: AD8001AN, Package_DIP:DIP-8_W7.62mm, symbol Amplifier_Operational:AD8001AN
- added C12, C13, C14, C15, C6, C7, C8: C, Capacitor_SMD:C_0805_2012Metric, symbol Device:C
- added Q3: MMDT3946, Package_TO_SOT_SMD:SOT-363_SC-70-6, symbol Transistor_BJT:MMDT3946
- added R10, R11, R12, R15, R9: R, Resistor_SMD:R_0805_2012Metric, symbol Device:R
- added U2: LM386, Package_DIP:DIP-8_W7.62mm, symbol Amplifier_Audio:LM386
Connections:
- net +5V: now also R13.1, C13.2, C14.1, C15.1, R11.1, R9.1, U2.6 (V+)
- net AM_Out: now also C12.1
- net Feed_BackBFin: now also U2.3 (+)
- net GND: now also C13.1, C14.2, C15.2, C6.1, C8.2, Q3.1 (E1), R12.2, R15.2, U2.4 (GND)
- net H1: now also C8.1, Q3.4 (E2); no longer R13.1
- net W1: now also U2.2 (-)
- net at Q1.2 (B), Q2.2 (B): now also U2.5
- net at C4.1, R13.2, R14.1: now also Q3.2 (B1)
- new net: Q3.6 (C1), R10.1, R9.2
- new net: C12.2, Q3.3 (C2), R15.1
- new net: Q3.5 (B2), R10.2, R11.2, R12.1
- new net: C7.2, U2.1 (GAIN)
- new net: C6.2, U2.7 (BYPASS)
- new net: C7.1, U2.8 (GAIN)
Other:
- note removed: "AFT05MS003N"

Commit message: Schematics and PCB update
Other:
- note added: "MMDT5451-7-F"
Changed lines of the file:
@@
 Wire Wire Line
 	7750 3850 7750 4300
+Text Notes 8200 3700 0    50   ~ 0
+MMDT5451-7-F
 $EndSCHEMATC
